File: PCB/Navi_2_0.sch (KiCad schematic (older format))
At the start: 110 parts, among them J1 USB_B_Micro, J10 BAT-, J2 Conn_01x24_Male, J23 Conn_01x06_Male, J27 Micro_SD_Card_Det, J8 SELECT, J9 BAT+, Q1 DMG2301L-7, Q2 Q_NMOS_GSD, Q3 DMG2301L-7, Q6 DMG2301L-7, SW1 SW_Push, SW2 SW_Push, U1 MT3420C, U2 MT3420C, U3 ESP32-WROOM-32, U4 CH330N, U5 L96-M33, U6 LSM6DS3, U7 TCN75-3.3

Commit message: Meeeeehr Widerstand
Meeeeehr Widerstand (Test)
Parts:
- R18: value 4K7 -> 4K8
Changed lines of the file:
@@
 P 3450 3000
 F 0 "R18" V 3400 3150 50  0000 L CNN
-F 1 "4K7" V 3450 2900 50  0000 L CNN
+F 1 "4K8" V 3450 2900 50  0000 L CNN
 F 2 "Resistor_SMD:R_0603_1608Metric" V 3380 3000 50  0001 C CNN
 F 3 "~" H 3450 3000 50  0001 C CNN
